Commit message: Fix Ridgeback mesh issue.
We were using an outdated URDF. Now actually leverage the info in the
ridgeback_description package rather than using an old copied version.

File: mm_description/urdf/mm.urdf.xacro (robot description, xacro)
@@ -1,227 +1,6 @@
 <?xml version="1.0"?>
 <robot name="Thing" xmlns:xacro="http://ros.org/wiki/xacro">
-  <xacro:property name="PI" value="3.1415926535897931" />
-  <xacro:property name="wheel_radius" value="0.0759" />
-  <xacro:property name="wheel_width" value="0.0790" />
-  <xacro:property name="chassis_length" value="0.960" />
-  <xacro:property name="chassis_width" value="0.793" />
-  <xacro:property name="chassis_height" value="0.216" />
-  <xacro:property name="deck_height" value="0.280" />
-  <xacro:property name="axle_offset" value="0.0500" />
-  <xacro:property name="rocker_offset" value="0.319" />
-  <xacro:property name="rocker_width" value="0.472" />
-  <xacro:property name="imu_offset_x" value="0.2085" />
-  <xacro:property name="imu_offset_y" value="-0.2902" />
-  <xacro:property name="imu_offset_z" value="0.1681" />
-  <xacro:property name="dummy_inertia" value="1e-09"/>
-  <material name="dark_grey"><color rgba="0.2 0.2 0.2 1.0" /></material>
-  <material name="light_grey"><color rgba="0.4 0.4 0.4 1.0" /></material>
-  <material name="yellow"><color rgba="0.8 0.8 0.0 1.0" /></material>
-  <material name="black"><color rgba="0.15 0.15 0.15 1.0" /></material>
-  <xacro:macro name="wheel" params="prefix side *joint_pose">
-    <link name="${prefix}_${side}_wheel_link">
-      <visual>
-        <origin xyz="0 0 0" rpy="${PI/2} 0 0"/>
-        <geometry>
-          <mesh filename="package://ridgeback_description/meshes/wheel.stl"/>
-        </geometry>
-        <material name="black" />
-      </visual>
-      <collision>
-        <origin xyz="0 0 0" rpy="${PI/2} 0 0"/>
-        <geometry>
-          <cylinder radius="${wheel_radius}" length="${wheel_width}"/>
-        </geometry>
-      </collision>
-      <inertial>
-        <origin xyz="0 0 0" rpy="0 0 0"/>
-        <mass value="0.477"/>
-        <inertia
-          ixx="0.0013" ixy="0" ixz="0"
-          iyy="0.0024" iyz="0"
-          izz="0.0013"/>
-      </inertial>
-    </link>
-    <joint name="${prefix}_${side}_wheel" type="continuous">
-      <parent link="${prefix}_rocker_link"/>
-      <child link="${prefix}_${side}_wheel_link" />
-      <xacro:insert_block name="joint_pose" />
-      <axis xyz="0 1 0" />
-    </joint>
-    <transmission name="${prefix}_wheel_trans">
-      <type>transmission_interface/SimpleTransmission</type>
-      <joint name="${prefix}_${side}_wheel">
-        <hardwareInterface>VelocityJointInterface</hardwareInterface>
-      </joint>
-      <actuator name="${prefix}_${side}_actuator">
-        <mechanicalReduction>1</mechanicalReduction>
-      </actuator>
-    </transmission>
-  </xacro:macro>
-  <xacro:macro name="rocker" params="prefix joint_type location *joint_limits">
-    <link name="${prefix}_rocker_link">
-      <visual>
-        <origin xyz="0 0 0" rpy="${PI/2} 0 ${PI/2}" />
-        <geometry>
-          <mesh filename="package://ridgeback_description/meshes/rocker.stl"/>
-        </geometry>
-        <material name="black" />
-      </visual>
-      <inertial>
-        <origin xyz="0 0 0" rpy="0 0 0"/>
-        <mass value="3"/>
-        <inertia
-          ixx="0.001" ixy="0" ixz="0"
-          iyy="0.001" iyz="0"
-          izz="0.001"/>
-      </inertial>
-    </link>
-    <joint name="${prefix}_rocker" type="${joint_type}">
-      <parent link="axle_link"/>
-      <child link="${prefix}_rocker_link" />
-      <origin xyz="${location*rocker_offset} 0 0" rpy="0 0 0" />
-      <axis xyz="1 0 0" />
-      <xacro:insert_block name="joint_limits" />
-    </joint>
-    <xacro:wheel prefix="${prefix}" side="left">
-      <origin xyz="0 ${rocker_width/2 + wheel_width/2} 0" rpy="0 0 0" />
-    </xacro:wheel>
-    <xacro:wheel prefix="${prefix}" side="right">
-      <origin xyz="0 ${-(rocker_width/2 + wheel_width/2)} 0" rpy="0 0 0" />
-    </xacro:wheel>
-  </xacro:macro>
-  <!-- DISABLING (joint limits) FREE ROCKER FOR NOW BECAUSE ROBOT SLIDES WITH IT-->
-  <!--xacro:rocker prefix="front" joint_type="revolute" location="1" >
-    <limit lower="0.08726" upper="0.08726" position="0" effort="0" velocity="0" />
-  </xacro:rocker-->
-  <xacro:rocker prefix="front" joint_type="fixed" location="1" >
-    <limit effort="0" velocity="0" />
-  </xacro:rocker>
-  <xacro:rocker prefix="rear" joint_type="fixed" location="-1" >
-    <limit effort="0" velocity="0" />
-  </xacro:rocker>
-  <link name="base_link"></link>
-  <joint name="base_link_joint" type="fixed">
-    <origin xyz="0 0 0" rpy="0 0 0" />
-    <parent link="base_link"/>
-    <child link="chassis_link" />
-  </joint>
-  <link name="chassis_link">
-    <visual>
-      <origin xyz="0 0 0" rpy=" ${PI/2} 0 ${PI/2}" />
-      <geometry>
-        <mesh filename="package://ridgeback_description/meshes/body.stl"/>
-      </geometry>
-      <material name="black" />
-    </visual>
-    <collision>
-      <origin xyz="0 0 ${chassis_height/2}"/>
-      <geometry>
-        <box size="${chassis_length} ${chassis_width} ${chassis_height}"/>
-      </geometry>
-    </collision>
-    <inertial>
-      <origin xyz="0.012 0.002 0.067" rpy="0 0 0"/>
-      <mass value="50"/>
-      <inertia
-        ixx="1.3136" ixy="0.0" ixz="0.0"
-        iyy="1.3922" iyz="0.0"
-        izz="2.0"/>
-    </inertial>
-  </link>
-  <joint name="front_cover_link_joint" type="fixed">
-    <origin xyz="0 0 0" rpy="0 0 0" />
-    <parent link="chassis_link"/>
-    <child link="front_cover_link" />
-  </joint>
-  <link name="front_cover_link">
-    <visual>
-      <origin xyz="0 0 0" rpy=" ${PI/2} 0 ${-PI/2}"  />
-      <geometry>
-        <mesh filename="package://ridgeback_description/meshes/end-cover.stl" />
-      </geometry>
-      <material name="black" />
-    </visual>
-  </link>
-  <joint name="rear_cover_link_joint" type="fixed">
-    <origin xyz="0 0 0" rpy="0 0 0" />
-    <parent link="chassis_link"/>
-    <child link="rear_cover_link" />
-  </joint>
-  <link name="rear_cover_link">
-    <visual>
-      <origin xyz="0 0 0" rpy=" ${PI/2} 0 ${PI/2}"  />
-      <geometry>
-        <mesh filename="package://ridgeback_description/meshes/end-cover.stl" />
-      </geometry>
-      <material name="black" />
-    </visual>
-  </link>
-  <joint name="top_link_joint" type="fixed">
-    <origin xyz="0 0 0" rpy="0 0 0" />
-    <parent link="chassis_link"/>
-    <child link="top_link" />
-  </joint>
-  <link name="top_link">
-    <visual>
-      <origin xyz="${-chassis_length/2} ${-chassis_width/2} 0" rpy=" ${PI/2} 0 ${PI/2}" />
-      <geometry>
-        <mesh filename="package://ridgeback_description/meshes/top.stl" />
-      </geometry>
-      <material name="black" />
-    </visual>
-  </link>
-  <joint name="ridgeback_x" type="continuous">
-    <origin xyz="0 0 0" rpy="0 0 0" />
-    <parent link="chassis_link"/>
-    <child link="top_link2" />
-  </joint>
-  <joint name="ridgeback_y" type="continuous">
-    <origin xyz="0 0 0" rpy="0 0 0" />
-    <parent link="chassis_link"/>
-    <child link="top_link3" />
-  </joint>
-  <joint name="ridgeback_theta" type="continuous">
-    <origin xyz="0 0 0" rpy="0 0 0" />
-    <parent link="chassis_link"/>
-    <child link="top_link4" />
-  </joint>
-  <link name="top_link2" />
-  <link name="top_link3" />
-  <link name="top_link4" />
-  <joint name="axle_joint" type="fixed">
-    <origin xyz="0 0 ${axle_offset}" rpy="0 0 0" />
-    <parent link="chassis_link"/>
-    <child link="axle_link" />
-  </joint>
-  <link name="axle_link">
-    <visual>
-      <origin xyz="0 0 0" rpy="0 ${PI/2} 0" />
-      <geometry>
-        <mesh filename="package://ridgeback_description/meshes/axle.stl" />
-      </geometry>
-      <material name="black" />
-    </visual>
-  </link>
-  <link name="imu_link">
-    <inertial>
-      <mass value="0.001"/>
-      <origin xyz="0 0 0" rpy="0 0 0"/>
-      <inertia ixx="${dummy_inertia}" ixy="0.0" ixz="0.0" iyy="${dummy_inertia}" iyz="0.0" izz="${dummy_inertia}"/>
-    </inertial>
-  </link>
-  <joint name="imu_joint" type="fixed">
-    <parent link="chassis_link" />
-    <child link="imu_link" />
-    <origin xyz="${imu_offset_x} ${imu_offset_y} ${imu_offset_z}" rpy="0 0 0"/>
-  </joint>
-  <link name="mid_mount" />
-  <joint name="mid_mount_joint" type="fixed">
-    <parent link="base_link" />
-    <child link="mid_mount" />
-    <origin xyz="0 0 ${deck_height}" rpy="0 0 0"/>
-  </joint>
-  <!-- Bring in simulation data for Gazebo. -->
-  <xacro:include filename="$(find mm_description)/urdf/ridgeback.gazebo" />
+  <!-- Spawn Ridgeback -->
+  <xacro:include filename="$(find ridgeback_description)/urdf/ridgeback.urdf.xacro" />
   <!-- Spawn arch -->
   <link name="arch_link">
@@ -293,5 +72,5 @@
   <!--<xacro:s-model_articulated prefix="" />-->
 <!-- origin, may be worth fixing better later: .03m from center of .06 long FT sensor plus extra link pieces, palm is 104.8mm long so assuming frame is at 52.4mm, minus 9.5mm for coupling -->
-  <xacro:include filename="$(find robotiq_s_model_visualization)/cfg/robotiq_hand_macro.urdf.xacro" />
+  <xacro:include filename="$(find robotiq_3f_gripper_visualization)/cfg/robotiq_hand_macro.urdf.xacro" />
   <xacro:robotiq_hand prefix="l_" parent="ur10_arm_ee_link" reflect="-1">
     <origin xyz="0.11 0.0 0.0" rpy="0.0 ${PI/12} -${PI/2}"/>

Commit message: Better instructions; clean up description.
* Leverage more existing packages rather than duplicating their code in
  the URDF description.
* Update with instructions from a relatively fresh melodic install

File: mm_description/urdf/mm.urdf.xacro (robot description, xacro)
@@ -10,9 +10,9 @@
 			</geometry>
 		</visual>
-		<collision>
-			<geometry>
-				<mesh filename="package://mm_description/meshes/tor11_mech.dae" />
-			</geometry>
-		</collision>
+		<!-- <collision> -->
+		<!-- 	<geometry> -->
+		<!-- 		<mesh filename="package://mm_description/meshes/tor11_mech.dae" /> -->
+		<!-- 	</geometry> -->
+		<!-- </collision> -->
    </link>
   <joint name="arch_joint" type="fixed">
@@ -22,6 +22,6 @@
   </joint>
   <!-- Spawn UR10 arm -->
-  <xacro:include filename="$(find mm_description)/urdf/ur10.urdf.xacro" />
-  <xacro:ur10_robot prefix="ur10_arm_" joint_limited="false"/>
+  <xacro:include filename="$(find ur_description)/urdf/ur10.urdf.xacro" />
+  <xacro:ur10_robot prefix="ur10_arm_" joint_limited="false" transmission_hw_interface="hardware_interface/VelocityJointInterface"/>
   <!-- Tool frame -->
   <xacro:property name="TCP_offset" value="0.29" />  <!-- must also be changed in thing_kinematics.h if changed here -->
@@ -69,19 +69,19 @@
  	  <child link="wrist_cam_mount_link" />
    </joint>
-  <!-- Spawn and Join Gripper. Giving it a prefix of l_ to work with gazebo plugin -->
-  <!--<xacro:s-model_articulated prefix="" />-->
-<!-- origin, may be worth fixing better later: .03m from center of .06 long FT sensor plus extra link pieces, palm is 104.8mm long so assuming frame is at 52.4mm, minus 9.5mm for coupling -->
-  <xacro:include filename="$(find robotiq_3f_gripper_visualization)/cfg/robotiq_hand_macro.urdf.xacro" />
-  <xacro:robotiq_hand prefix="l_" parent="ur10_arm_ee_link" reflect="-1">
-    <origin xyz="0.11 0.0 0.0" rpy="0.0 ${PI/12} -${PI/2}"/>
-  </xacro:robotiq_hand>
-  <!-- gazebo for gripper -->
-   <gazebo>
-    <plugin name="robotiq_hand_plugin" filename="libRobotiqHandPlugin.so">
-      <side>left</side>
-      <kp_position>10.0</kp_position>
-      <kd_position>0.5</kd_position>
-    </plugin>
-  </gazebo>
+   <!-- origin, may be worth fixing better later: .03m from center of .06 long FT sensor plus extra link pieces, palm is 104.8mm long so assuming frame is at 52.4mm, minus 9.5mm for coupling -->
+   <!-- TODO: gripper disabled for now because it seems to cause weird dynamic in Gazebo -->
+  <!-- <xacro:include filename="$(find robotiq_3f_gripper_visualization)/cfg/robotiq_hand_macro.urdf.xacro" /> -->
+  <!-- <xacro:robotiq_hand prefix="l_" parent="ur10_arm_ee_link" reflect="&#45;1"> -->
+  <!--   <origin xyz="0.11 0.0 0.0" rpy="0.0 ${PI/12} &#45;${PI/2}"/> -->
+  <!-- </xacro:robotiq_hand> -->
+  <!--  -->
+  <!-- <!&#45;&#45; gazebo for gripper &#45;&#45;> -->
+  <!--  <gazebo> -->
+  <!--   <plugin name="robotiq_hand_plugin" filename="libRobotiqHandPlugin.so"> -->
+  <!--     <side>left</side> -->
+  <!--     <kp_position>10.0</kp_position> -->
+  <!--     <kd_position>0.5</kd_position> -->
+  <!--   </plugin> -->
+  <!-- </gazebo> -->
   <!-- Inflate collision geometry near connectors-->
   <!--
